File: subsystems/experimental/mobility/eagle/main_brd.brd (EAGLE design)
At the start: 207.7 x 178.7 mm, 91 parts, among them IC1 74LS245DW

Commit message: mobility vhdl project updated
Parts:
- removed BTN: (no value), switch-misc:RACON12
- removed IC1: 74LS245DW, 74xx-us:SO20W
- removed J3: (no value), con-jack:SPC4077
- removed R14, R15, R16: 10k, resistor:R1206
- removed SW_1, SW_2, SW_3: (no value), switch:TL3XPO
- removed U$6: TPD2E2U06DRLR, ti-esd:DRL5
- added C1, C11, C24, C29, C30, C51, C6: 1nF, rcl:C1206
- added C12, C13, C14, C15, C16, C17, C18, C19, C20, C21: (no value), rcl:C1206
- added C2, C7: 0.1uF, rcl:C1206
- added C22, C23: 1uF, resistor:E1,8-4
- added ENC_0, ENC_1, ENC_2, ENC_3, ENC_4, ENC_5, ENC_6, ENC_7, ENC_8, ENC_9, US_0, US_1, US_2, US_3, US_4, US_5, US_6, US_7: (no value), con-lstb:MA04-1
- added ENC_PR_0_A, ENC_PR_0_B, ENC_PR_1_A, ENC_PR_1_B, ENC_PR_2_A, ENC_PR_2_B, ENC_PR_3_A, ENC_PR_3_B, ENC_PR_4_A, ENC_PR_4_B, ENC_PR_5_A, ENC_PR_5_B, ENC_PR_6_A, ENC_PR_6_B, ENC_PR_7_A, ENC_PR_7_B, ENC_PR_8_A, ENC_PR_8_B, ENC_PR_9_A, ENC_PR_9_B, US_PR_0, US_PR_1, US_PR_2, US_PR_3, US_PR_4, US_PR_5, US_PR_6, US_PR_7: (no value), resistor:R1206
- added LEFT, REAR, RIGHT, STEER_L, STEER_R: (no value), con-subd:F25HP
- added R10, R36, R5, R6, R7, R8, R9: 22, resistor:R1206
- added R17: 51, resistor:R1206
- added SV14, SV15, SV16, SV17, SV4, SV5, SV6: (no value), con-lstb:MA03-1
- added SV18: (no value), con-lstb:MA03-2
- added U$10, U$11, U$9: ADC128S052QCMT, kamal:R-PDSO-G16
- added U$7, U$8: MB02-1, kamal:MB03-1
- C26: value 10uf -> 1nF; device resistor:C1206 -> rcl:C1206
- R2: value 10k -> 22
- SV2: device con-lstb:MA04-2 -> con-lstb:MA03-1
- moved C26 152.7 mm to (117.5, -21.0)
- moved SW_0 124.8 mm to (219.1, 62.9), turned to 0 degrees
- moved SV3 108.4 mm to (-31.8, -1.27), turned to 0 degrees
- moved R1 105.6 mm to (63.5, 77.5)
- moved RST 67.3 mm to (62.9, 74.3)
- moved R2 66.3 mm to (62.9, -40.6), turned to 90 degrees
- moved SV2 63.1 mm to (142.2, -8.26), turned to 90 degrees
- moved U$4 62.1 mm to (65.4, 73.0)
- moved C32 58.5 mm to (7.59, 62.6), turned to 0 degrees
- moved U$1 58.3 mm to (-19.7, 102.9)
- moved SV1 58.3 mm to (-14.6, 100.3)
- moved U$5 58.3 mm to (-19.7, 98.4)
- moved C31 56.7 mm to (7.59, 58.6), turned to 0 degrees
- moved C28 55.8 mm to (12.5, 69.4), turned to 270 degrees
- moved C34 55.5 mm to (7.59, 54.4), turned to 0 degrees
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Connections:
- net ENC_A_0 renamed 97
- net ENC_A_1 renamed 95
- net ENC_B_0 renamed 98
- net ENC_B_1 renamed 96
- removed net 57: 37_TO_72.21
- removed net 58: 37_TO_72.22
- removed net 59: 37_TO_72.23
- removed net 60: 37_TO_72.24
- removed net 66: 37_TO_72.30
- removed net 67: 37_TO_72.31
- removed net 68: 37_TO_72.32
- removed net 70: 37_TO_72.34
- removed net 72: 37_TO_72.36
- removed net BTN_1: 1_TO_36.7, IC1.11
- removed net ENC_A_2: 73_TO_108.21
- removed net ENC_A_3: 73_TO_108.16
- removed net ENC_A_4: 73_TO_108.14
- removed net ENC_A_5: 73_TO_108.12
- removed net ENC_A_6: 73_TO_108.8
- removed net ENC_A_7: 73_TO_108.5
- removed net ENC_A_8: 73_TO_108.3
- removed net ENC_A_9: 73_TO_108.1
- removed net ENC_B_2: 73_TO_108.22
- removed net ENC_B_3: 73_TO_108.19
- removed net ENC_B_4: 73_TO_108.15
- removed net ENC_B_5: 73_TO_108.13
- removed net ENC_B_6: 73_TO_108.9
- removed net ENC_B_7: 73_TO_108.7
- removed net ENC_B_8: 73_TO_108.4
- removed net ENC_B_9: 73_TO_108.2
- removed net EN_2: 37_TO_72.1
- removed net EN_3: 37_TO_72.15
- removed net EN_7: 37_TO_72.4
- removed net EN_8: 37_TO_72.7
- removed net EN_9: 37_TO_72.12
- removed net PWM_F_2: 37_TO_72.2
- removed net PWM_F_3: 37_TO_72.16
- removed net PWM_F_7: 37_TO_72.5
- removed net PWM_F_8: 37_TO_72.8
- removed net PWM_F_9: 37_TO_72.13
- removed net PWM_R_2: 37_TO_72.3
- removed net PWM_R_3: 37_TO_72.17
- removed net PWM_R_7: 37_TO_72.6
- removed net PWM_R_8: 37_TO_72.9
- removed net PWM_R_9: 37_TO_72.14
- removed net SS_H_2: 37_TO_72.19
- new net 0_A: ENC_0.3, ENC_PR_0_A.2
- new net 0_B: ENC_0.4, ENC_PR_0_B.2
- new net 101: 73_TO_108.29
- new net 102: 73_TO_108.30
- new net 103: 73_TO_108.31
- new net 104: 73_TO_108.32
- new net 105: 73_TO_108.33
- new net 106: 73_TO_108.34
- new net 107: 73_TO_108.35
- new net 108: 73_TO_108.36
- new net 123: 144_TO_109.15
- new net 13: 1_TO_36.13
- new net 1_A: ENC_1.3, ENC_PR_1_A.2
- new net 1_B: ENC_1.4, ENC_PR_1_B.2
- new net 2_A: ENC_2.3, ENC_PR_2_A.2
- new net 2_B: ENC_2.4, ENC_PR_2_B.2
- new net 3_A: ENC_3.3, ENC_PR_3_A.2
- new net 3_B: ENC_3.4, ENC_PR_3_B.2
- new net 4_A: ENC_4.3, ENC_PR_4_A.2
- new net 4_B: ENC_4.4, ENC_PR_4_B.2
- new net 5_A: ENC_5.3, ENC_PR_5_A.2
- new net 5_B: ENC_5.4, ENC_PR_5_B.2
- new net 6_A: ENC_6.3, ENC_PR_6_A.2
- new net 6_B: ENC_6.4, ENC_PR_6_B.2
- new net 7_A: ENC_7.3, ENC_PR_7_A.2
- new net 7_B: ENC_7.4, ENC_PR_7_B.2
- new net 8_A: ENC_8.3, ENC_PR_8_A.2
- new net 8_B: ENC_8.4, ENC_PR_8_B.2
- new net 9_A: ENC_9.3, ENC_PR_9_A.2
- new net 9_B: ENC_9.4, ENC_PR_9_B.2
- new net CS_FL: LEFT.17
- new net CS_FR: RIGHT.17
- new net CS_ML: LEFT.19
- new net CS_MR: RIGHT.19
- new net CS_RL: REAR.17
- new net CS_RR: REAR.19
- new net D1_FL: 37_TO_72.16, LEFT.4
- new net D1_FR: RIGHT.4
- new net D1_ML: 37_TO_72.12, LEFT.6
- new net D1_MR: RIGHT.6
- new net D1_RL: 37_TO_72.35, REAR.4
- new net D1_RR: 37_TO_72.31, REAR.6
- new net D2_FL: 37_TO_72.15, LEFT.16
- new net D2_FR: RIGHT.16
- new net D2_ML: 37_TO_72.14, LEFT.18
- new net D2_MR: RIGHT.18
- new net D2_RL: 37_TO_72.36, REAR.16
- new net D2_RR: 37_TO_72.34, REAR.18
- new net ENC_0_A: ENC_PR_0_A.1
- new net ENC_0_B: ENC_PR_0_B.1
- new net ENC_1_A: ENC_PR_1_A.1
- new net ENC_1_B: ENC_PR_1_B.1
- new net ENC_2_A: ENC_PR_2_A.1
- new net ENC_2_B: ENC_PR_2_B.1
- new net ENC_3_A: ENC_PR_3_A.1
- new net ENC_3_B: ENC_PR_3_B.1
- new net ENC_4_A: ENC_PR_4_A.1
- new net ENC_4_B: ENC_PR_4_B.1
- new net ENC_5_A: 73_TO_108.1, ENC_PR_5_A.1
- new net ENC_5_B: 73_TO_108.2, ENC_PR_5_B.1
- new net ENC_6_A: 73_TO_108.9, ENC_PR_6_A.1
- new net ENC_6_B: 73_TO_108.7, ENC_PR_6_B.1
- new net ENC_7_A: 73_TO_108.3, ENC_PR_7_A.1
- new net ENC_7_B: 73_TO_108.4, ENC_PR_7_B.1
- new net ENC_8_A: 73_TO_108.8, ENC_PR_8_A.1
- new net ENC_8_B: 73_TO_108.5, ENC_PR_8_B.1
- new net ENC_9_A: ENC_PR_9_A.1
- new net ENC_9_B: ENC_PR_9_B.1
- new net E_0: US_0.3, US_PR_0.2
- new net E_1: US_1.3, US_PR_1.2
- new net E_2: US_2.3, US_PR_2.2
- new net E_3: US_3.3, US_PR_3.2
- new net E_4: US_4.3, US_PR_4.2
- new net E_5: US_5.3, US_PR_5.2
- new net E_6: US_6.3, US_PR_6.2
- new net E_7: US_7.3, US_PR_7.2
- new net IN0: C11.1, U$9.4
- new net IN1: C1.1, U$9.5
- new net IN2: C6.1, U$9.6
- new net IN3: C24.1, U$9.7
- new net IN4: C26.1, U$9.8
- new net IN5: C29.1, U$9.9
- new net IN6: C30.1, U$9.10
- new net IN7: C51.1, U$9.11
- new net N$15: R6.1
- new net N$4: C18.1, C20.2
- new net N$5: R2.1
- new net N$69: R6.2
- new net N$7: R8.1
- new net N$70: R5.2
- new net N$71: R9.2
- new net N$72: R8.2
- new net N$73: R2.2
- new net N$74: R10.1
- new net N$76: R36.1
- new net N$77: R10.2
- new net N$79: R36.2
- new net N$8: R9.1
- new net N$9: R5.1
- new net POT_0: SV14.2
- new net POT_1: SV15.2
- new net POT_2: SV16.2
- new net POT_3: SV17.2
- new net PWM_FL: 37_TO_72.13, LEFT.5
- new net PWM_FR: RIGHT.5
- new net PWM_ML: 37_TO_72.9, LEFT.7
- new net PWM_MR: RIGHT.7
- new net PWM_RL: 37_TO_72.33, REAR.5
- new net PWM_RR: 37_TO_72.32, REAR.7
- new net SCS_FL: STEER_L.17
- new net SCS_FR: STEER_R.17
- new net SCS_RL: STEER_L.19
- new net SCS_RR: STEER_R.19
- new net SD1_FL: 37_TO_72.5, STEER_L.4
- new net SD1_FR: STEER_R.4
- new net SD1_RL: 37_TO_72.4, STEER_L.6
- new net SD1_RR: STEER_R.6
- new net SD2_FL: 37_TO_72.8, STEER_L.16
- new net SD2_FR: STEER_R.16
- new net SD2_RL: 37_TO_72.3, STEER_L.18
- new net SD2_RR: STEER_R.18
- new net SPWM_FL: 37_TO_72.6, STEER_L.5
- new net SPWM_FR: STEER_R.5
- new net SPWM_RL: 37_TO_72.1, STEER_L.7
- new net SPWM_RR: STEER_R.7
- new net SS_H_3: 37_TO_72.30, REAR.11
- new net SS_H_4: 37_TO_72.7, LEFT.11
- new net SS_H_5: RIGHT.11
- new net SS_H_6: 37_TO_72.2, STEER_L.11
- new net SS_H_7: STEER_R.11
- new net V24_D: LEFT.1, LEFT.14, LEFT.15, LEFT.2, REAR.1, REAR.14, REAR.15, REAR.2, RIGHT.1, RIGHT.14, RIGHT.15, RIGHT.2, U$8.1
- new net V24_S: STEER_L.1, STEER_L.14, STEER_L.15, STEER_L.2, STEER_R.1, STEER_R.14, STEER_R.15, STEER_R.2, U$7.1
- new net VA: C2.1, C22.+, R17.2, U$9.2
- new net VD: C23.+, C7.1, R17.1, U$9.13
- net BTN: no longer BTN.1, BTN.2, C26.1, IC1.9
- net BTN_0: no longer IC1.12
- net EN_0: now also 144_TO_109.21; no longer 144_TO_109.22
- net EN_4: now also 144_TO_109.24; no longer 144_TO_109.25
- net EN_6: now also 144_TO_109.31; no longer 144_TO_109.33
- net GND: now also C1.2, C11.2, C2.2, C22.-, C23.-, C7.2, ENC_0.2, ENC_1.2, ENC_2.2, ENC_3.2, ENC_4.2, ENC_5.2, ENC_6.2, ENC_7.2, ENC_8.2, ENC_9.2, LEFT.12, LEFT.13, LEFT.24, LEFT.25, LEFT.3, LEFT.G1, LEFT.G2, REAR.12, REAR.13, REAR.24, REAR.25, REAR.3, REAR.G1, REAR.G2, RIGHT.12, RIGHT.13, RIGHT.24, RIGHT.25, RIGHT.3, RIGHT.G1, RIGHT.G2, STEER_L.12, STEER_L.13, STEER_L.24, STEER_L.25, STEER_L.3, STEER_L.G1, STEER_L.G2, STEER_R.12, STEER_R.13, STEER_R.24, STEER_R.25, STEER_R.3, STEER_R.G1, STEER_R.G2, SV14.3, SV15.3, SV16.3, SV17.3, SV18.5, SV18.6, U$7.2, U$8.2, U$9.12, U$9.3, US_0.4, US_1.4, US_2.4, US_3.4, US_4.4, US_5.4, US_6.4, US_7.4; no longer BTN.3, BTN.4, C25.2, C26.2, IC1.10, IC1.19, J3.1, SV2.3, SV2.4, SW_1.3, SW_2.3, SW_3.3
- net MISO_H: now also 144_TO_109.12, 37_TO_72.22, LEFT.9, REAR.9, RIGHT.9, STEER_L.9, STEER_R.9, U$9.15; no longer 144_TO_109.15
- net MOSI_H: now also 144_TO_109.11, 37_TO_72.21, LEFT.21, REAR.21, RIGHT.21, STEER_L.21, STEER_R.21, U$9.14; no longer 144_TO_109.14
- net N$30: now also R7.1; no longer R14.1, SW_1.2
- net N$31: now also C24.2, C26.2, C29.2, C30.2, C51.2, C6.2; no longer R15.1, SW_2.2
- net N$32: now also R7.2; no longer R16.1, SW_3.2
- net PWM_F_0: now also 144_TO_109.22; no longer 144_TO_109.21
- net PWM_F_4: now also 144_TO_109.25; no longer 144_TO_109.24
- net PWM_F_6: now also 144_TO_109.34; no longer 144_TO_109.32
- net PWM_R_1: now also 144_TO_109.33; no longer 144_TO_109.34
- net PWM_R_6: now also 144_TO_109.32; no longer 144_TO_109.31
- net RST: now also R1.1; no longer IC1.8
- net RX: no longer SV2.1
- net SCK_H: now also 144_TO_109.14, 37_TO_72.24, LEFT.22, REAR.22, RIGHT.22, STEER_L.22, STEER_R.22, U$9.16; no longer 144_TO_109.13
- net SCL_H: now also 37_TO_72.17, LEFT.23, REAR.23, RIGHT.23, STEER_L.23, STEER_R.23; no longer 37_TO_72.33
- net SDA_H: now also 37_TO_72.19, LEFT.10, REAR.10, RIGHT.10, STEER_L.10, STEER_R.10; no longer 37_TO_72.35
- net SS_H_0: now also 144_TO_109.13; no longer 144_TO_109.12
- net SS_H_1: now also 37_TO_72.23, U$9.1; no longer 144_TO_109.11
- net SW_0: now also 1_TO_36.7; no longer 1_TO_36.13
- net SW_1: no longer R14.2
- net SW_2: no longer R15.2
- net SW_3: no longer R16.2
- net TCK: now also SV18.3; no longer SV2.8
- net TDI: now also SV18.2; no longer SV2.5
- net TDO: now also SV18.4; no longer SV2.7
- net TMS: now also SV18.1; no longer SV2.6
- net TX: no longer SV2.2
- net US_E_0: now also 73_TO_108.21, US_PR_0.1; no longer 73_TO_108.36
- net US_E_1: now also 73_TO_108.13, US_PR_1.1; no longer 73_TO_108.35
- net US_E_2: now also 73_TO_108.14, US_PR_2.1; no longer 73_TO_108.34
- net US_E_3: now also 73_TO_108.12, US_PR_3.1; no longer 73_TO_108.33
- net US_E_4: now also 73_TO_108.22, US_PR_4.1; no longer 73_TO_108.32
- net US_E_5: now also 73_TO_108.16, US_PR_5.1; no longer 73_TO_108.31
- net US_E_6: now also 73_TO_108.15, US_PR_6.1; no longer 73_TO_108.30
- net US_E_7: now also 73_TO_108.19, US_PR_7.1; no longer 73_TO_108.29
- net US_T_0: now also 144_TO_109.2, US_0.2; no longer 144_TO_109.10
- net US_T_1: now also 144_TO_109.1, US_1.2; no longer 144_TO_109.9
- net US_T_2: now also 144_TO_109.4, US_2.2; no longer 144_TO_109.6
- net US_T_3: now also 144_TO_109.3, US_3.2; no longer 144_TO_109.5
- net US_T_4: now also 144_TO_109.9, US_4.2; no longer 144_TO_109.4
- net US_T_5: now also 144_TO_109.10, US_5.2; no longer 144_TO_109.3
- net US_T_6: now also 144_TO_109.5, US_6.2; no longer 144_TO_109.2
- net US_T_7: now also 144_TO_109.6, US_7.2; no longer 144_TO_109.1
- net VCC: now also ENC_0.1, ENC_1.1, ENC_2.1, ENC_3.1, ENC_4.1, ENC_5.1, ENC_6.1, ENC_7.1, ENC_8.1, ENC_9.1, SV14.1, SV15.1, SV16.1, SV17.1, US_0.1, US_1.1, US_2.1, US_3.1, US_4.1, US_5.1, US_6.1, US_7.1
- net VCCIO: now also LEFT.20, LEFT.8, R1.2, REAR.20, REAR.8, RIGHT.20, RIGHT.8, STEER_L.20, STEER_L.8, STEER_R.20, STEER_R.8; no longer IC1.1, IC1.20, SW_1.1, SW_2.1, SW_3.1
- net VIN: no longer J3.3
Routing:
- net VCCIO: track 220.1 -> 476.5 mm, vias 3 -> 7
- net SCK_H: track 0.00 -> 222.8 mm, vias 0 -> 5
- net MOSI_H: track 0.00 -> 221.4 mm, vias 0 -> 3
- net MISO_H: track 0.00 -> 202.0 mm, vias 0 -> 3
- net SCL_H: track 0.00 -> 201.5 mm, vias 0 -> 5
- net SDA_H: track 0.00 -> 194.4 mm, vias 0 -> 5
- net V24_D: track 0.00 -> 167.1 mm
- net SDA_S: track 150.8 -> 0.00 mm, vias 2 -> 0
- net SCL_S: track 143.0 -> 5.13 mm, vias 3 -> 0
- net US_T_1: track 0.00 -> 135.0 mm
- net US_T_5: track 0.00 -> 133.8 mm
- net US_T_2: track 0.00 -> 126.8 mm
- net US_T_6: track 0.00 -> 120.4 mm
- net US_T_3: track 0.00 -> 118.5 mm
- net VCC: track 13.5 -> 126.1 mm
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- removed copper zone on layer 1, net GND
- removed copper zone on layer 16, net GND
Other:
- board size 207.7 x 178.7 mm -> 194.4 x 120.3 mm
